File: Electronics/Schematics/PIL/pil.kicad_pcb (KiCad board)
At the start: 2 copper layers, 20 parts

Commit message: update all
Parts:
- added ?: CAM_RX_TX, Wire_Pads:SolderWirePad_2x_0-8mmDrill, F.Cu at (80.0, 91.4)
- added ?: GND_3.3, Wire_Pads:SolderWirePad_2x_0-8mmDrill, F.Cu at (57.1, 143.5)
- added ?: , Resistors_ThroughHole:Resistor_Horizontal_RM10mm, F.Cu at (34.3, 139.7)
- added ?: DA_CL, Wire_Pads:SolderWirePad_2x_0-8mmDrill, F.Cu at (49.5, 143.5)
- added ?: , Wire_Pads:SolderWirePad_4xInline_0-8mmDrill, F.Cu at (33.0, 127.0)
- added ? (x2): , Wire_Pads:SolderWirePad_4xInline_0-8mmDrill, F.Cu at (33.0, 90.2)
- added ?: , Wire_Pads:SolderWirePad_4xInline_0-8mmDrill, F.Cu at (33.0, 76.2)
- added ?: G_RX_TX, Wire_Pads:SolderWirePad_2x_0-8mmDrill, F.Cu at (41.9, 143.5)
- added ?: , Wire_Pads:SolderWirePad_3x_0-8mmDrill, F.Cu at (81.3, 39.4)
- added ?: , Wire_Pads:SolderWirePad_4xInline_0-8mmDrill, F.Cu at (92.7, 59.7)
- added ?: GND_3.3, Wire_Pads:SolderWirePad_2x_0-8mmDrill, F.Cu at (80.0, 143.5)
- added ?: CAM_-_5.0, Wire_Pads:SolderWirePad_2x_0-8mmDrill, F.Cu at (61.0, 91.4)
- added ?: SOLAR Out, Wire_Pads:SolderWirePad_2x_0-8mmDrill, F.Cu at (69.8, 143.5)
- added ?: TMP OUT, Wire_Pads:SolderWirePad_2x_0-8mmDrill, F.Cu at (68.6, 16.5)
- added ?: UV Out, Wire_Pads:SolderWirePad_2x_0-8mmDrill, F.Cu at (45.7, 38.1)
- added ?: , Resistors_ThroughHole:Resistor_Horizontal_RM10mm, F.Cu at (49.5, 22.9)
- added ?: 5.0, Wire_Pads:SolderWirePad_2x_0-8mmDrill, F.Cu at (63.5, 143.5)
- added ?: , Resistors_ThroughHole:Resistor_Horizontal_RM10mm, F.Cu at (24.1, 139.7)
- added ADXL345: ADX1, Wire_Pads:SolderWirePad_4xInline_0-8mmDrill, F.Cu at (33.0, 76.2)
- added BMP180: BMP1, Wire_Pads:SolderWirePad_4xInline_0-8mmDrill, F.Cu at (33.0, 54.6)
- added ML8511: ML1, Wire_Pads:SolderWirePad_4xInline_0-8mmDrill, F.Cu at (33.0, 27.9)
- added RHT03: RH1, Wire_Pads:SolderWirePad_4xInline_0-8mmDrill, F.Cu at (63.5, 27.9)
- added SD Card: SD1, Wire_Pads:SolderWirePad_4xInline_0-8mmDrill, F.Cu at (81.3, 27.9)
- added SPARKFUN_VENUS_GPS: GPS1, Wire_Pads:SolderWirePad_4xInline_0-8mmDrill, F.Cu at (33.0, 113.0)
- added SP_215: PY1, Wire_Pads:SolderWirePad_3x_0-8mmDrill, F.Cu at (68.6, 54.6)
- moved LM1 76.2 mm to (144.1, 80.3)
- moved LM1 76.2 mm to (187.1, 80.3)
- moved LM1 76.2 mm to (187.1, 29.3)
- moved LM1 76.2 mm to (144.1, 29.3)
- moved R1 76.2 mm to (140.3, 90.5)
- moved R1 76.2 mm to (183.3, 90.5)
- moved R1 76.2 mm to (183.3, 39.5)
- moved R1 76.2 mm to (140.3, 39.5)
- moved IN 76.2 mm to (174.4, 75.2)
- moved IN 76.2 mm to (174.4, 24.2)
- moved OUT 76.2 mm to (174.4, 103.2)
- moved OUT 76.2 mm to (174.4, 52.2)
- moved IN 76.2 mm to (131.4, 75.2)
- moved IN 76.2 mm to (131.4, 24.2)
- moved OUT 76.2 mm to (131.4, 103.2)
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Routing:
- net (no net): track 471.0 -> 2331.7 mm

Commit message: update kicad files
Parts:
- moved ? 38.7 mm to (128.3, 74.9)
- moved ? 38.7 mm to (85.1, 158.8)
- moved ? 38.7 mm to (77.5, 158.8)
- moved ? 38.7 mm to (116.8, 54.6)
- moved ? 38.7 mm to (105.4, 158.8)
- moved ? 38.7 mm to (104.1, 31.8)
- moved ? 38.7 mm to (81.3, 53.3)
- moved ? 38.7 mm to (85.1, 38.1)
- moved ? 38.7 mm to (99.1, 158.8)
- moved ? 38.7 mm to (59.7, 154.9)
- moved IN 38.7 mm to (167.0, 90.5)
- moved IN 38.7 mm to (210.0, 90.5)
- moved IN 38.7 mm to (210.0, 39.5)
- moved IN 38.7 mm to (167.0, 39.5)
- moved OUT 38.7 mm to (167.0, 118.4)
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
Commit message: extra fixes
Parts:
- removed the ? at (115.6, 106.7)
- removed the ? at (92.7, 158.8)
- removed the ? at (69.8, 154.9)
- removed the ? at (85.1, 158.8)
- removed the ? at (68.6, 142.2)
- removed the ? at (77.5, 158.8)
- removed the ? at (128.3, 74.9)
- removed the ? at (115.6, 158.8)
- removed the ? at (96.5, 106.7)
- removed the ? at (105.4, 158.8)
- removed the ? at (104.1, 31.8)
- removed the ? at (81.3, 53.3)
- removed the ? at (85.1, 38.1)
- removed the ? at (99.1, 158.8)
- removed the ? at (59.7, 154.9)
- removed IN (x4): In, Wire_Pads:SolderWirePad_2x_0-8mmDrill
- removed LM1 (x4): LM317, Wire_Pads:SolderWirePad_3x_1mmDrill
- removed OUT (x4): Out, Wire_Pads:SolderWirePad_2x_0-8mmDrill
- removed the R1 at (175.9, 105.7)
- removed the R1 at (218.9, 105.7)
- removed the R1 at (218.9, 54.7)
- removed the R1 at (175.9, 54.7)
- removed R2 (x4): 680Ω, Resistors_ThroughHole:Resistor_Horizontal_RM10mm
- removed SPARKFUN_VENUS_GPS: GPS1, Wire_Pads:SolderWirePad_4xInline_0-8mmDrill
- added ?: , Wire_Pads:SolderWirePad_4xInline_0-8mmDrill, F.Cu at (99.7, 111.1)
- added ?: , Wire_Pads:SolderWirePad_4xInline_0-8mmDrill, F.Cu at (60.3, 155.6)
- added ?: , Wire_Pads:SolderWirePad_4xInline_0-8mmDrill, F.Cu at (64.1, 155.6)
- added ?: , Wire_Pads:SolderWirePad_4xInline_0-8mmDrill, F.Cu at (67.9, 155.6)
- added ?: , Wire_Pads:SolderWirePad_4xInline_0-8mmDrill, F.Cu at (71.8, 155.6)
- added ?: , Wire_Pads:SolderWirePad_4xInline_0-8mmDrill, F.Cu at (95.9, 111.1)
- added ?: , Wire_Pads:SolderWirePad_4xInline_0-8mmDrill, F.Cu at (94.6, 104.8)
- added ?: , Wire_Pads:SolderWirePad_4xInline_0-8mmDrill, F.Cu at (75.6, 155.6)
- added R1: 1K, Resistors_ThroughHole:Resistor_Horizontal_RM10mm, F.Cu at (58.4, 63.5)
- added REF**: SolderWirePad_4xInline_1-2mmDrill, Wire_Pads:SolderWirePad_4xInline_1-2mmDrill, F.Cu at (120.7, 111.8)
- added REF**: SolderWirePad_4xInline_1-2mmDrill, Wire_Pads:SolderWirePad_4xInline_1-2mmDrill, F.Cu at (120.7, 108.0)
- added REF**: SolderWirePad_4xInline_1-2mmDrill, Wire_Pads:SolderWirePad_4xInline_1-2mmDrill, F.Cu at (120.7, 104.1)
- added REF**: SolderWirePad_4xInline_1-2mmDrill, Wire_Pads:SolderWirePad_4xInline_1-2mmDrill, F.Cu at (120.7, 95.2)
- added REF**: SolderWirePad_4xInline_1-2mmDrill, Wire_Pads:SolderWirePad_4xInline_1-2mmDrill, F.Cu at (120.7, 77.5)
- added REF**: SolderWirePad_4xInline_1-2mmDrill, Wire_Pads:SolderWirePad_4xInline_1-2mmDrill, F.Cu at (120.7, 86.4)
- moved ML8511 147.7 mm to (215.9, 53.3)
- moved SP_215 98.1 mm to (200.7, 52.1)
- moved ? 75.0 mm to (191.8, 57.1)
- moved SD Card 75.0 mm to (191.8, 45.7)
- moved RHT03 28.7 mm to (78.7, 63.5), turned to 0 degrees
- moved ? 18.0 mm to (81.9, 93.3), turned to 180 degrees (x2)
- moved BMP180 13.3 mm to (81.3, 73.7), turned to 180 degrees
- moved ? 2.01 mm to (67.9, 93.3), turned to 180 degrees
- moved ADXL345 2.01 mm to (67.9, 93.3), turned to 180 degrees
Routing:
- net (no net): track 2331.7 -> 468.3 mm

Commit message: Final Launch Code!
Parts:
- added REF**: SolderWirePad_single_0-8mmDrill, Wire_Pads:SolderWirePad_single_0-8mmDrill, F.Cu at (111.8, 111.8)
- added REF**: SolderWirePad_single_0-8mmDrill, Wire_Pads:SolderWirePad_single_0-8mmDrill, F.Cu at (111.8, 108.0)
- added REF**: SolderWirePad_single_0-8mmDrill, Wire_Pads:SolderWirePad_single_0-8mmDrill, F.Cu at (111.8, 104.1)
- added REF**: SolderWirePad_single_0-8mmDrill, Wire_Pads:SolderWirePad_single_0-8mmDrill, F.Cu at (111.8, 95.2)
- added REF**: SolderWirePad_single_0-8mmDrill, Wire_Pads:SolderWirePad_single_0-8mmDrill, F.Cu at (111.8, 86.4)
- added REF**: SolderWirePad_single_0-8mmDrill, Wire_Pads:SolderWirePad_single_0-8mmDrill, F.Cu at (111.8, 77.5)
Routing:
- net (no net): track 468.3 -> 494.9 mm
Changed lines of the file:
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@@
     (thickness 1.6)
     (drawings 0)
-    (tracks 44)
+    (tracks 50)
     (zones 0)
-    (modules 25)
+    (modules 31)
     (nets 1)
   )
@@
   )
   (setup
-    (last_trace_width 0.25)
+    (last_trace_width 2)
     (user_trace_width 1)
     (user_trace_width 2)
@@
     (mod_text_size 1 1)
     (mod_text_width 0.15)
-    (pad_size 1.99898 1.99898)
-    (pad_drill 0.8001)
+    (pad_size 2.99974 2.99974)
+    (pad_drill 1.19888)
     (pad_to_mask_clearance 0.2)
     (aux_axis_origin 0 0)
@@
     (uvia_drill 0.1)
   )
+  (module Wire_Pads:SolderWirePad_single_0-8mmDrill (layer F.Cu)
+    (at 111.76 111.76)
+    (fp_text reference REF** (at 0 -2.54) (layer F.SilkS)
+      (effects (font (size 1 1) (thickness 0.15)))
+    )
+    (fp_text value SolderWirePad_single_0-8mmDrill (at 0 2.54) (layer F.Fab)
+      (effects (font (size 1 1) (thickness 0.15)))
+    )
+    (pad 1 thru_hole circle (at -1.27 0) (size 2.99974 2.99974) (drill 1.19888) (layers *.Cu *.Mask F.SilkS))
+  )
+  (module Wire_Pads:SolderWirePad_single_0-8mmDrill (layer F.Cu)
+    (at 111.76 107.95)
+    (fp_text reference REF** (at 0 -2.54) (layer F.SilkS)
+      (effects (font (size 1 1) (thickness 0.15)))
+    )
+    (fp_text value SolderWirePad_single_0-8mmDrill (at 0 2.54) (layer F.Fab)
+      (effects (font (size 1 1) (thickness 0.15)))
+    )
+    (pad 1 thru_hole circle (at -1.27 0) (size 2.99974 2.99974) (drill 1.19888) (layers *.Cu *.Mask F.SilkS))
+  )
+  (module Wire_Pads:SolderWirePad_single_0-8mmDrill (layer F.Cu)
+    (at 111.76 104.14)
+    (fp_text reference REF** (at 0 -2.54) (layer F.SilkS)
+      (effects (font (size 1 1) (thickness 0.15)))
+    )
+    (fp_text value SolderWirePad_single_0-8mmDrill (at 0 2.54) (layer F.Fab)
+      (effects (font (size 1 1) (thickness 0.15)))
+    )
+    (pad 1 thru_hole circle (at -1.27 0) (size 2.99974 2.99974) (drill 1.19888) (layers *.Cu *.Mask F.SilkS))
+  )
+  (module Wire_Pads:SolderWirePad_single_0-8mmDrill (layer F.Cu)
+    (at 111.76 95.25)
+    (fp_text reference REF** (at 0 -2.54) (layer F.SilkS)
+      (effects (font (size 1 1) (thickness 0.15)))
+    )
+    (fp_text value SolderWirePad_single_0-8mmDrill (at 0 2.54) (layer F.Fab)
+      (effects (font (size 1 1) (thickness 0.15)))
+    )
+    (pad 1 thru_hole circle (at -1.27 0) (size 2.99974 2.99974) (drill 1.19888) (layers *.Cu *.Mask F.SilkS))
+  )
+  (module Wire_Pads:SolderWirePad_single_0-8mmDrill (layer F.Cu)
+    (at 111.76 86.36)
+    (fp_text reference REF** (at 0 -2.54) (layer F.SilkS)
+      (effects (font (size 1 1) (thickness 0.15)))
+    )
+    (fp_text value SolderWirePad_single_0-8mmDrill (at 0 2.54) (layer F.Fab)
+      (effects (font (size 1 1) (thickness 0.15)))
+    )
+    (pad 1 thru_hole circle (at -1.27 0) (size 2.99974 2.99974) (drill 1.19888) (layers *.Cu *.Mask F.SilkS))
+  )
+  (module Wire_Pads:SolderWirePad_single_0-8mmDrill (layer F.Cu)
+    (at 111.76 77.47)
+    (fp_text reference REF** (at 0 -2.54) (layer F.SilkS)
+      (effects (font (size 1 1) (thickness 0.15)))
+    )
+    (fp_text value SolderWirePad_single_0-8mmDrill (at 0 2.54) (layer F.Fab)
+      (effects (font (size 1 1) (thickness 0.15)))
+    )
+    (pad 1 thru_hole circle (at -1.27 0) (size 2.99974 2.99974) (drill 1.19888) (layers *.Cu *.Mask F.SilkS))
+  )
   (module Wire_Pads:SolderWirePad_4xInline_1-2mmDrill (layer F.Cu)
     (at 120.65 111.76)
@@
     (pad 1 thru_hole circle (at 5.715 0) (size 2.99974 2.99974) (drill 1.19888) (layers *.Cu *.Mask F.SilkS))
   )
+  (segment (start 110.49 86.36) (end 114.935 86.36) (width 2) (layer B.Cu) (net 0) (status C00000))
+  (segment (start 110.49 95.25) (end 114.935 95.25) (width 2) (layer B.Cu) (net 0) (status C00000))
+  (segment (start 110.49 107.95) (end 110.49 111.76) (width 2) (layer B.Cu) (net 0) (status C00000))
+  (segment (start 110.49 111.76) (end 114.935 111.76) (width 2) (layer B.Cu) (net 0) (status C00000))
+  (segment (start 110.49 107.95) (end 114.935 107.95) (width 2) (layer B.Cu) (net 0) (status C00000))
+  (segment (start 110.49 104.14) (end 114.935 104.14) (width 2) (layer B.Cu) (net 0) (status C00000))
+  (segment (start 110.49 77.47) (end 114.935 77.47) (width 2) (layer B.Cu) (net 0))
   (segment (start 114.935 104.14) (end 126.365 104.14) (width 2) (layer B.Cu) (net 0))
   (segment (start 126.365 104.14) (end 126.365 107.95) (width 2) (layer B.Cu) (net 0))
   (segment (start 126.365 107.95) (end 114.935 107.95) (width 2) (layer B.Cu) (net 0))
-  (segment (start 114.935 107.95) (end 114.935 111.76) (width 2) (layer B.Cu) (net 0))
   (segment (start 114.935 111.76) (end 126.365 111.76) (width 2) (layer B.Cu) (net 0))
   (segment (start 114.935 95.25) (end 126.365 95.25) (width 2) (layer B.Cu) (net 0))
